File: STM32 PCB/STM32 PCB.kicad_pcb (KiCad board)
At the start: 2 copper layers, 2 parts, among them U1 NUCLEO-L476RG

Commit message: PCB upload
Parts:
- added J1: Screw_Terminal_01x15, Connector_PinSocket_2.54mm:PinSocket_1x15_P2.54mm_Vertical, F.Cu at (225.2, 116.8)
- added J3: Conn_01x08_Pin, Connector_PinSocket_2.54mm:PinSocket_1x08_P2.54mm_Vertical, F.Cu at (178.5, 34.7)

Commit message: KiCad PCB
Routing:
- added copper zone on B.Cu, net GND
Changed lines of the file:
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@@
 	)
 	(setup
+		(stackup
+			(layer "F.SilkS"
+				(type "Top Silk Screen")
+			)
+			(layer "F.Paste"
+				(type "Top Solder Paste")
+			)
+			(layer "F.Mask"
+				(type "Top Solder Mask")
+				(thickness 0.01)
+			)
+			(layer "F.Cu"
+				(type "copper")
+				(thickness 0.035)
+			)
+			(layer "dielectric 1"
+				(type "core")
+				(thickness 1.51)
+				(material "FR4")
+				(epsilon_r 4.5)
+				(loss_tangent 0.02)
+			)
+			(layer "B.Cu"
+				(type "copper")
+				(thickness 0.035)
+			)
+			(layer "B.Mask"
+				(type "Bottom Solder Mask")
+				(thickness 0.01)
+			)
+			(layer "B.Paste"
+				(type "Bottom Solder Paste")
+			)
+			(layer "B.SilkS"
+				(type "Bottom Silk Screen")
+			)
+			(copper_finish "None")
+			(dielectric_constraints no)
+		)
 		(pad_to_mask_clearance 0)
 		(allow_soldermask_bridges_in_footprints no)
@@
 			)
 		)
+	)
+	(zone
+		(net 1)
+		(net_name "GND")
+		(layer "B.Cu")
+		(hatch edge 0.5)
+		(connect_pads
+			(clearance 0.5)
+		)
+		(min_thickness 0.25)
+		(filled_areas_thickness no)
+		(fill
+			(thermal_gap 0.5)
+			(thermal_bridge_width 0.5)
+		)
+		(polygon
+			(pts
+				(xy 89.2 17.35) (xy 271.8 17.2) (xy 276.85 158.15) (xy 88.55 157.25)
+			)
+		)

Commit message: PCB updates
Parts:
- added C1: 1 uF, Capacitor_SMD:C_0805_2012Metric_Pad1.18x1.45mm_HandSolder, F.Cu at (207.6, 48.7)
- added J10: Conn_01x03_Socket, Connector_PinHeader_2.54mm:PinHeader_1x03_P2.54mm_Vertical, F.Cu at (207.5, 84.9)
- added J2: Conn_01x03_Socket, Connector_PinHeader_2.54mm:PinHeader_1x03_P2.54mm_Vertical, F.Cu at (207.5, 120.0)
- added J4: Conn_01x03_Socket, Connector_PinHeader_2.54mm:PinHeader_1x03_P2.54mm_Vertical, F.Cu at (207.5, 70.0)
- added J5: Conn_01x03_Socket, Connector_PinHeader_2.54mm:PinHeader_1x03_P2.54mm_Vertical, F.Cu at (220.6, 58.1)
- added J6: Conn_01x03_Socket, Connector_PinHeader_2.54mm:PinHeader_1x03_P2.54mm_Vertical, F.Cu at (127.5, 70.0)
- added J7: Conn_01x03_Socket, Connector_PinHeader_2.54mm:PinHeader_1x03_P2.54mm_Vertical, F.Cu at (127.5, 90.0)
- added J8: Conn_01x03_Socket, Connector_PinHeader_2.54mm:PinHeader_1x03_P2.54mm_Vertical, F.Cu at (127.5, 105.0)
- added J9: Conn_01x03_Socket, Connector_PinHeader_2.54mm:PinHeader_1x03_P2.54mm_Vertical, F.Cu at (127.5, 120.1)
- J1: value Screw_Terminal_01x15 -> Conn_01x03_Socket; footprint Connector_PinSocket_2.54mm:PinSocket_1x15_P2.54mm_Vertical -> Connector_PinHeader_2.54mm:PinHeader_1x03_P2.54mm_Vertical
- J3: value Conn_01x08_Pin -> Conn_01x03_Socket; footprint Connector_PinSocket_2.54mm:PinSocket_1x08_P2.54mm_Vertical -> Connector_PinHeader_2.54mm:PinHeader_1x03_P2.54mm_Vertical
- R1: value 100 -> 1000 ohm; footprint Resistor_THT:R_Axial_DIN0411_L9.9mm_D3.6mm_P12.70mm_Horizontal -> Resistor_SMD:R_0805_2012Metric_Pad1.20x1.40mm_HandSolder
- moved R1 104.0 mm to (207.6, 43.3)
- moved J3 76.1 mm to (207.5, 105.1), turned to 180 degrees
- moved J1 64.3 mm to (207.5, 55.0), turned to 0 degrees
Connections:
- J1 pad 1: YPUL -> GND
- J1 pad 2: YEN -> unconnected-(J1-Pin_2-Pad2)
- J1 pad 3: YDIR -> Vin
- J3 pad 1: SPI1_CD -> XPUL
- J3 pad 2: SPI1_CS -> XEN
- J3 pad 3: SPI_MOSI -> XDIR
- R1 pad 1: shutdownButton -> Net-(U1A-PA1)
- R1 pad 2: GND -> Out of Bounds -
- U1 pad CN10_16: unconnected-(U1B-PB12-PadCN10_16) -> GPIO_PB12
- U1 pad CN10_17: SPI1_CS -> SPI_CS
- U1 pad CN10_18: unconnected-(U1B-PB11-PadCN10_18) -> GPIO_PB11
- U1 pad CN10_19: SPI1_CD -> SPI_CD
- U1 pad CN10_21: YDIR -> XDIR
- U1 pad CN10_23: YEN -> XEN
- U1 pad CN10_25: YPUL -> XPUL
- U1 pad CN10_27: XDIR -> YDIR
- U1 pad CN10_28: unconnected-(U1B-PB14-PadCN10_28) -> GPIO_PB14
- U1 pad CN10_29: XEN -> YEN
- U1 pad CN10_3: unconnected-(U1B-PB8-PadCN10_3) -> I2C_SDL
- U1 pad CN10_30: unconnected-(U1B-PB13-PadCN10_30) -> GPIO_PB13
- U1 pad CN10_33: XPUL -> YPUL
- U1 pad CN7_16: +3V3 -> Out of Bounds +
- U1 pad CN7_18: +5V -> 5V
- U1 pad CN7_21: unconnected-(U1A-PB7-PadCN7_21) -> I2C_SDA
- U1 pad CN7_24: VCC -> Vin
- U1 pad CN7_30: shutdownButton -> Net-(U1A-PA1)
- U1 pad CN7_32: unconnected-(U1A-PA4-PadCN7_32) -> btn0
- U1 pad CN7_34: unconnected-(U1A-PB0-PadCN7_34) -> btn1
- U1 pad CN7_35: unconnected-(U1A-PC2-PadCN7_35) -> btn4
- U1 pad CN7_36: unconnected-(U1A-PC1-PadCN7_36) -> btn2
- U1 pad CN7_38: unconnected-(U1A-PC0-PadCN7_38) -> btn3
Routing:
- net GPIO_PB11: track 0.00 -> 84.3 mm
- net GPIO_PB14: track 0.00 -> 33.4 mm
- net GPIO_PB13: track 0.00 -> 30.9 mm
- net SPI_CD: track 0.00 -> 24.8 mm
- net SPI_CS: track 0.00 -> 24.7 mm
- net SPI_MOSI: track 0.00 -> 24.7 mm
- net Out of Bounds +: track 0.00 -> 22.8 mm
- net 5V: track 0.00 -> 22.3 mm
- net Laser_PWM: track 0.00 -> 21.1 mm
- net YEN: track 0.00 -> 16.8 mm
- net YDIR: track 0.00 -> 16.3 mm
- net btn0: track 0.00 -> 15.6 mm
- net I2C_SDA: track 0.00 -> 15.5 mm
- net btn2: track 0.00 -> 15.3 mm
- net btn1: track 0.00 -> 15.3 mm
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
Commit message: kiCad final board upload
Parts:
- moved R1 81.5 mm to (127.7, 59.2), turned to 180 degrees
- moved C1 81.4 mm to (127.6, 64.0), turned to 180 degrees
- moved J5 14.8 mm to (207.5, 65.0)
- moved J4 7.46 mm to (207.5, 77.4)
- moved J10 5.04 mm to (207.5, 90.0)
- moved J1 2.58 mm to (207.5, 52.4)
- moved J3 2.42 mm to (207.5, 107.5)
Routing:
- net I2C_SDL: track 0.00 -> 195.7 mm
- net Vin: track 0.00 -> 86.9 mm
- net Net-(U1A-PA1): track 0.00 -> 63.2 mm
- net GND: track 0.14 -> 39.0 mm
- net SPI_MISO: track 0.00 -> 22.0 mm
- net SPI_SCK: track 0.00 -> 21.9 mm
- net Out of Bounds -: track 0.00 -> 12.0 mm
- net SPI_MOSI: track 24.7 -> 17.2 mm
- net SPI_CS: track 24.7 -> 17.3 mm
- net SPI_CD: track 24.8 -> 18.7 mm
- net GPIO_PB12: track 8.69 -> 10.8 mm
- net XPUL: track 12.2 -> 13.2 mm
- net XDIR: track 12.2 -> 13.2 mm
- net XEN: track 12.2 -> 13.2 mm
- net GPIO_PB13: track 30.9 -> 29.9 mm
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Other:
- board outline added: 103.8 x 86.3 mm
- board text added: "5V"
- board text added: "GND"
- board text added: "GPIO"
- board text added: "I2C_SDA"
- board text added: "I2C_SDL"
- board text added: "Laser_PWM"
- board text added: "Out of Bounds+"
- board text added: "Out of Bounds-"
- board text added: "SPI CD"
- board text added: "SPI CS"
- board text added: "SPI MISO"
- board text added: "SPI MOSI"
- board text added: "SPI SCK"
- board text added: "Vin"
- board text added: "XDIR"
- board text added: "XEN"
- board text added: "XPUL"
- board text added: "YDIR"
- board text added: "YEN"
- board text added: "YPUL"
- board text added: "btn0"
- board text added: "btn1"
- board text added: "btn2"
- board text added: "btn3"
- board text added: "btn4"
